File: kicad/lna.kicad_sch (KiCad schematic)
At the start: 34 parts, among them J4 Conn_01x02_Pin, J5 Conn_Coaxial_Small, J6 Conn_Coaxial_Small, U5 L78L05_SOT89, U6 BFP640, U7 BFP640, U8 BFP640

Commit message: files ready for production, but with wrong stackup (3313)
Parts:
- removed C18: 2.2nF, Capacitor_SMD:C_0805_2012Metric, symbol Device:C_Small
- added C4, C7: 100pF, Capacitor_SMD:C_0402_1005Metric, symbol Device:C_Small
- Z3, Z6, Z7: now not fitted
Connections:
- net +5V: now also C4.1
- net GND: now also C4.2, C7.2
- net at R14.2, R15.1: now also C7.1
Other:
- moved on the sheet: C14

Commit message: placed jlcpcb order, waiting for gerber confirmation
Parts:
- Z2: LCSC Part Number C76953 -> C1550; Manufacturing Part Number GRM1555C1H1R0CA01D -> 0402CG1R0C500NT
Changed lines of the file:
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@@
 			)
 		)
-		(property "Datasheet" "https://wmsc.lcsc.com/wmsc/upload/file/pdf/v2/lcsc/1811081611_Murata-Electronics-GRM1555C1H1R0CA01D_C76953.pdf"
+		(property "Datasheet" "https://www.lcsc.com/datasheet/lcsc_datasheet_2304140030_FH--Guangdong-Fenghua-Advanced-Tech-0402CG1R0C500NT_C1550.pdf"
 			(at 133.35 120.65 0)
 			(effects
@@
 			)
 		)
-		(property "LCSC Part Number" "C76953"
+		(property "LCSC Part Number" "C1550"
 			(at 133.35 120.65 0)
 			(effects
@@
 			)
 		)
-		(property "Manufacturing Part Number" "GRM1555C1H1R0CA01D"
+		(property "Manufacturing Part Number" "0402CG1R0C500NT"
 			(at 133.35 120.65 0)
 			(effects
