File: kicad/rf_lna.kicad_sch (KiCad schematic)
At the start: 0 parts

Commit message: placed jlcpcb order, waiting for gerber confirmation
Parts:
- added FID1, FID2, FID3: Fiducial, Fiducial:Fiducial_1mm_Mask2mm, symbol Mechanical:Fiducial
- added H1, H2, H3, H4: MountingHole, antennas:MountingHole_1.152mm_jlcpcb, symbol Mechanical:MountingHole
