File: kicad/transistor.kicad_sch (KiCad schematic)
At the start: 28 parts, among them J1 Conn_01x02_Pin, J2 Conn_Coaxial_Small, J3 Conn_Coaxial_Small, U1 L78L05_SOT89, U3 BFP640

Commit message: placed jlcpcb order, waiting for gerber confirmation
Parts:
- Z12, Z8, Z9: LCSC Part Number C76953 -> C1550; Manufacturing Part Number GRM1555C1H1R0CA01D -> 0402CG1R0C500NT
Changed lines of the file:
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@@
 			)
 		)
-		(property "Datasheet" "https://wmsc.lcsc.com/wmsc/upload/file/pdf/v2/lcsc/1811081611_Murata-Electronics-GRM1555C1H1R0CA01D_C76953.pdf"
+		(property "Datasheet" "https://www.lcsc.com/datasheet/lcsc_datasheet_2304140030_FH--Guangdong-Fenghua-Advanced-Tech-0402CG1R0C500NT_C1550.pdf"
 			(at 151.13 95.25 0)
 			(effects
@@
 			)
 		)
-		(property "LCSC Part Number" "C76953"
+		(property "LCSC Part Number" "C1550"
 			(at 151.13 95.25 0)
 			(effects
@@
 			)
 		)
-		(property "Manufacturing Part Number" "GRM1555C1H1R0CA01D"
+		(property "Manufacturing Part Number" "0402CG1R0C500NT"
 			(at 151.13 95.25 0)
 			(effects
@@
 			)
 		)
-		(property "Datasheet" "https://wmsc.lcsc.com/wmsc/upload/file/pdf/v2/lcsc/1811081611_Murata-Electronics-GRM1555C1H1R0CA01D_C76953.pdf"
+		(property "Datasheet" "https://www.lcsc.com/datasheet/lcsc_datasheet_2304140030_FH--Guangdong-Fenghua-Advanced-Tech-0402CG1R0C500NT_C1550.pdf"
 			(at 224.79 88.9 0)
 			(effects
@@
 			)
 		)
-		(property "LCSC Part Number" "C76953"
+		(property "LCSC Part Number" "C1550"
 			(at 224.79 88.9 0)
 			(effects
@@
 			)
 		)
-		(property "Manufacturing Part Number" "GRM1555C1H1R0CA01D"
+		(property "Manufacturing Part Number" "0402CG1R0C500NT"
 			(at 224.79 88.9 0)
 			(effects
@@
 			)
 		)
-		(property "Datasheet" "https://wmsc.lcsc.com/wmsc/upload/file/pdf/v2/lcsc/1811081611_Murata-Electronics-GRM1555C1H1R0CA01D_C76953.pdf"
+		(property "Datasheet" "https://www.lcsc.com/datasheet/lcsc_datasheet_2304140030_FH--Guangdong-Fenghua-Advanced-Tech-0402CG1R0C500NT_C1550.pdf"
 			(at 246.38 88.9 0)
 			(effects
@@
 			)
 		)
-		(property "LCSC Part Number" "C76953"
+		(property "LCSC Part Number" "C1550"
 			(at 246.38 88.9 0)
 			(effects
@@
 			)
 		)
-		(property "Manufacturing Part Number" "GRM1555C1H1R0CA01D"
+		(property "Manufacturing Part Number" "0402CG1R0C500NT"
 			(at 246.38 88.9 0)
 			(effects
